File: eagle/Mecanumbot Power Board/Mecanumbot Power Board.sch (EAGLE design)
At the start: 99 parts, among them J1 AVR_SPI_PRG_6PTH, U1 FT232RL-BASICSSOP, U2 ATMEGA168, X1 USBSMD, Y1 RESONATORSMD

Commit message: pushing back v2.0 from svn
Parts:
- removed C12, C13, C14, C17, C2, C3, C6: 1uF, SparkFun:CAP0603-CAP
- removed C15, C22, C4: 0.1uF, SparkFun:CAP0603-CAP
- removed C16, C5: 330uF, SparkFun:CAP_POL3528
- removed C18: 68uF, SparkFun:CAP_POL1206
- removed JP4: FIDUCIAL1X2.5, SparkFun:FIDUCIAL1X2.5
- removed JP6: PWR LED, SparkFun:M02PTH
- removed R10: 24K, SparkFun:RESISTOR0603-RES
- removed R11, R8: 1K, SparkFun:RESISTOR0603-RES
- removed R22: 10K, SparkFun:RESISTOR0603-RES
- removed R26: 3.3K, SparkFun:RESISTOR0603-RES
- removed R35, R36: 10k, SparkFun:RESISTOR0603-RES
- removed R5: 7.5K, SparkFun:RESISTOR0603-RES
- removed R9: 200K, SparkFun:RESISTOR0603-RES
- removed U$15, U$9: TERMINAL-4MINIFIT-JR, AT-Parts-RJ:TERMINAL-4MINIFIT-JR
- removed U$21: SUPERCAPS-LEAD, AT-Parts-RJ:SUPERCAPS-LEAD
- removed U$22: HMC6352, SparkFun:HMC6352
- added PC-CTRL: S2, SparkFun:M02PTH
- JP2: value FIDUCIAL1X2.5 -> USB; device SparkFun:FIDUCIAL1X2.5 -> SparkFun:M04PTH
- JP3: value FIDUCIAL1X2.5 -> PWR-CTRL; device SparkFun:FIDUCIAL1X2.5 -> SparkFun:M04PTH
- LED3: value Green -> Yellow
- LED4, LED5, LED6: value RED -> Blue; device SparkFun:LED5MM -> SparkFun:LED0603
- R37: value 10k -> 10K
- R4: value 7.5K -> 330
- R6: value 200K -> 10K
- R7: value 24K -> 3.3K
- U$1: value IR3477 -> CLA230TR-NDSMD; device AT-Parts-RJ:IR3477 -> jav-parts:CLA230TR-NDSMD
- U$2, U$4: value 1uH -> BZT52C33-FDICT-ND; device SparkFun:INDUCTORPWR -> jav-parts:BZT52C33-FDICT-ND
- U$3: value IR3477 -> BZT52C33-FDICT-ND; device AT-Parts-RJ:IR3477 -> jav-parts:BZT52C33-FDICT-ND
Connections:
- removed net 12VA: C19.+, C21.1, C5.+, R22.2, R7.2, U$15.3, U$15.4, U$17.3, U$17.4, U$19.EN, U$19.IN, U$2.2, U$21.P$1
- removed net 12VB: C16.+, R10.2, U$16.3, U$16.4, U$4.2
- removed net N$17: R4.1, U$3.ISET
- removed net N$18: C3.2, U$1.3VCBP
- removed net N$19: R6.1, U$1.FF
- removed net N$21: R10.1, R11.2, U$3.FB
- removed net N$22: C14.2, U$3.3VCBP
- removed net N$23: R9.1, U$3.FF
- removed net N$24: C15.2, U$3.SS
- removed net N$25: C4.2, U$1.SS
- removed net N$35: R19.2, U2.PD6(AIN0)
- removed net N$36: R20.2, U2.PD5(T1)
- removed net N$37: R21.2, U2.PD3(INT1)
- removed net N$41: R22.1, R26.2, U2.PC3(ADC3)
- removed net N$45: JP6.1, R30.2
- removed net POST-DIODE: U$11.P$2, U$5.P$2, U$8.P$2, U$9.1, U$9.2
- new net N$14: R20.2, U2.PB2(SS/OC1B)
- new net PCCTRL: R4.1, U2.PB0(ICP)
- new net PWRSW: JP3.4, R6.2, U$2.CA, U$3.CA, U$4.CA
- net BATT1EN: now also U2.PD6(AIN0); no longer U2.PB0(ICP)
- net BATT2EN: now also U2.PD5(T1); no longer U2.PB1(OC1A)
- net GND: now also JP2.1, JP3.2, JP3.3, R7.1, S1.2, U$1.CTRL-; no longer C12.2, C13.2, C14.1, C15.1, C16.-, C18.-, C2.2, C22.2, C3.1, C4.1, C5.-, JP6.2, R11.1, R26.1, R8.1, S1.1, U$1.FCCM, U$1.GND, U$1.GND1, U$1.PGND, U$15.1, U$15.2, U$21.P$2, U$22.GND, U$3.FCCM, U$3.GND, U$3.GND1, U$3.PGND
- net MOSI: now also R21.2
- net N$12: now also R4.2, U$1.CTRL+; no longer R5.1, U$1.ISET
- net N$13: now also JP3.1, R30.2; no longer C17.1, U$3.BOOT
- net N$15: now also R33.2, R34.1, U2.PC3(ADC3); no longer C17.2, R4.2, U$3.PHASE, U$4.1
- net N$16: now also R19.2, U2.PB1(OC1A); no longer R7.1, R8.2, U$1.FB
- net N$26: now also U$3.AN
- net N$29: now also U$2.AN
- net N$32: now also U$4.AN
- net N$42: now also U2.PC2(ADC2); no longer U2.PC0(ADC0)
- net N$44: now also U2.PC0(ADC0); no longer U2.PC2(ADC2)
- net N$46: now also R6.1, R7.2; no longer R33.2, R34.1
- net N$5: now also PC-CTRL.2, U$1.DC-; no longer C6.1, U$1.BOOT
- net N$6: now also PC-CTRL.1, U$1.DC+; no longer C6.2, R5.2, U$1.PHASE, U$2.1
- net N$7: now also JP2.3
- net N$8: now also JP2.2
- net PRE-VIN: now also U$11.P$2, U$5.P$2, U$8.P$2; no longer U$9.3, U$9.4
- net RESET: now also S1.1; no longer S1.2
- net SCL: no longer R35.1, U$22.SCL
- net SDA: no longer R36.1, U$22.SDA
- net VCC: now also JP2.4; no longer C13.1, C2.1, C22.1, R35.2, R36.2, U$1.EN, U$1.VCC, U$22.VCC, U$3.EN, U$3.VCC
- net VIN: now also C19.+, C21.1, U$16.3, U$16.4, U$17.3, U$17.4, U$19.EN, U$19.IN; no longer C12.1, C18.+, R6.2, R9.2, U$1.VIN, U$3.VIN
- net WALLPWREN: now also U2.PD7(AIN1); no longer U2.PB2(SS/OC1B)
Other:
- note added: "2"
- note added: "PC Control"
- note removed: "(Everything Else)"
- note removed: "(Motors)"
- note removed: "1"
- note removed: "12V Power A"
- note removed: "12V Power B"
- note removed: "Compass"
- moved on the sheet: C10, C7, C8, J1, JP1, JP7, LED1, LED2, LED3, LED4, LED5, LED6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
